Commit message: gazewbo and rviz  with LDF preload in my ubuntu

File: urdf/dummy_robot.urdf (robot description, URDF)
Before this commit: robot dummy_robot, 2 links, 1 joints
Links:
- link base_link: geometry visual box size=0.1 0.1 0.1
Joints:
- removed joint odom_to_base_link
- added joint odom_to_base: type fixed, parent odom, child base_link, origin xyz=0 0 0 rpy=0 0 0
